Commit message: added qbhand to curi robot and fixed material problem

File: urdf/curi.urdf (robot description, URDF)
Before this commit: robot curi, 35 links, 34 joints
Links:
- added link left_root_link
- added link qbhand_base_link, mass 0.205; collision mesh filename=../meshes/qbhand/flange_iso_04.stl scale=0.001 0.001 0.001; visual mesh filename=../meshes/qbhand/flange_iso_04.stl scale=0.001 0.001 0.001
- added link qbhand_end_effector_link
- added link qbhand_index_distal_link, mass 0.009; collision mesh filename=../meshes/qbhand/ph_distal_collision.stl scale=0.001 0.001 0.001; visual mesh filename=../meshes/qbhand/ph_distal.stl scale=0.001 0.001 0.001
- added link qbhand_index_distal_virtual_link, mass 1e-4
- added link qbhand_index_knuckle_link, mass 0.0095; collision mesh filename=../meshes/qbhand/ph_knuckle_collision.stl scale=0.001 0.001 0.001; visual mesh filename=../meshes/qbhand/meshes/ph_knuckle.stl scale=0.001 0.001 0.001
- added link qbhand_index_middle_link, mass 0.0063; collision mesh filename=../meshes/qbhand/ph_short_collision.stl scale=0.001 0.001 0.001; visual mesh filename=../meshes/qbhand/ph_short.stl scale=0.001 0.001 0.001
- added link qbhand_index_middle_virtual_link, mass 1e-4
- added link qbhand_index_proximal_link, mass 0.0082; collision mesh filename=../meshes/qbhand/ph_medium_collision.stl scale=0.001 0.001 0.001; visual mesh filename=../meshes/qbhand/ph_medium.stl scale=0.001 0.001 0.001
- added link qbhand_index_proximal_virtual_link, mass 1e-4
- added link qbhand_little_distal_link, mass 0.009; collision mesh filename=../meshes/qbhand/ph_distal_collision.stl scale=0.001 0.001 0.001; visual mesh filename=../meshes/qbhand/ph_distal.stl scale=0.001 0.001 0.001
- added link qbhand_little_distal_virtual_link, mass 1e-4
- added link qbhand_little_knuckle_link, mass 0.0095; collision mesh filename=../meshes/qbhand/ph_knuckle_collision.stl scale=0.001 0.001 0.001; visual mesh filename=../meshes/qbhand/ph_knuckle.stl scale=0.001 0.001 0.001
- added link qbhand_little_middle_link, mass 0.0063; collision mesh filename=../meshes/qbhand/ph_short_collision.stl scale=0.001 0.001 0.001; visual mesh filename=../meshes/qbhand/ph_short.stl scale=0.001 0.001 0.001
- added link qbhand_little_middle_virtual_link, mass 1e-4
- added link qbhand_little_proximal_link, mass 0.0063; collision mesh filename=../meshes/qbhand/ph_short_collision.stl scale=0.001 0.001 0.001; visual mesh filename=../meshes/qbhand/ph_short.stl scale=0.001 0.001 0.001
- added link qbhand_little_proximal_virtual_link, mass 1e-4
- added link qbhand_middle_distal_link, mass 0.009; collision mesh filename=../meshes/qbhand/ph_distal_collision.stl scale=0.001 0.001 0.001; visual mesh filename=../meshes/qbhand/ph_distal.stl scale=0.001 0.001 0.001
- added link qbhand_middle_distal_virtual_link, mass 1e-4
- added link qbhand_middle_knuckle_link, mass 0.0095; collision mesh filename=../meshes/qbhand/ph_knuckle_collision.stl scale=0.001 0.001 0.001; visual mesh filename=../meshes/qbhand/ph_knuckle.stl scale=0.001 0.001 0.001
- added link qbhand_middle_middle_link, mass 0.0063; collision mesh filename=../meshes/qbhand/ph_short_collision.stl scale=0.001 0.001 0.001; visual mesh filename=../meshes/qbhand/ph_short.stl scale=0.001 0.001 0.001
- added link qbhand_middle_middle_virtual_link, mass 1e-4
- added link qbhand_middle_proximal_link, mass 0.0082; collision mesh filename=../meshes/qbhand/ph_medium_collision.stl scale=0.001 0.001 0.001; visual mesh filename=../meshes/qbhand/ph_medium.stl scale=0.001 0.001 0.001
- added link qbhand_middle_proximal_virtual_link, mass 1e-4
- added link qbhand_palm_link, mass 0.45; collision mesh filename=../meshes/qbhand/palm_pinch_l.stl scale=0.001 0.001 0.001; visual mesh filename=../meshes/qbhand/palm_pinch_l.stl scale=0.001 0.001 0.001
- added link qbhand_ring_distal_link, mass 0.009; collision mesh filename=../meshes/qbhand/ph_distal_collision.stl scale=0.001 0.001 0.001; visual mesh filename=../meshes/qbhand/ph_distal.stl scale=0.001 0.001 0.001
- added link qbhand_ring_distal_virtual_link, mass 1e-4
- added link qbhand_ring_knuckle_link, mass 0.0095; collision mesh filename=../meshes/qbhand/ph_knuckle_collision.stl scale=0.001 0.001 0.001; visual mesh filename=../meshes/qbhand/ph_knuckle.stl scale=0.001 0.001 0.001
- added link qbhand_ring_middle_link, mass 0.0063; collision mesh filename=../meshes/qbhand/ph_short_collision.stl scale=0.001 0.001 0.001; visual mesh filename=../meshes/qbhand/ph_short.stl scale=0.001 0.001 0.001
- added link qbhand_ring_middle_virtual_link, mass 1e-4
- added link qbhand_ring_proximal_link, mass 0.0082; collision mesh filename=../meshes/qbhand/ph_medium_collision.stl scale=0.001 0.001 0.001; visual mesh filename=../meshes/qbhand/ph_medium.stl scale=0.001 0.001 0.001
- added link qbhand_ring_proximal_virtual_link, mass 1e-4
- added link qbhand_synergy_tendon_virtual_link, mass 1e-4
- added link qbhand_thumb_distal_link, mass 0.009; collision mesh filename=../meshes/qbhand/ph_distal_collision.stl scale=0.001 0.001 0.001; visual mesh filename=../meshes/qbhand/ph_distal.stl scale=0.001 0.001 0.001
- added link qbhand_thumb_distal_virtual_link, mass 1e-4
- added link qbhand_thumb_knuckle_link, mass 0.01; collision mesh filename=../meshes/qbhand/ph_thumb_l_collision.stl scale=0.001 0.001 0.001; visual mesh filename=../meshes/qbhand/ph_thumb_l.stl scale=0.001 0.001 0.001
- added link qbhand_thumb_proximal_link, mass 0.0063; collision mesh filename=../meshes/qbhand/ph_short_collision.stl scale=0.001 0.001 0.001; visual mesh filename=../meshes/qbhand/ph_short.stl scale=0.001 0.001 0.001
- added link qbhand_thumb_proximal_virtual_link, mass 1e-4
Joints:
- added joint panda_end_effector_joint: type fixed, parent panda_left_link7, child left_root_link, origin xyz=0 0 0.107 rpy=0 0 -0.7853981633974483
- added joint qbhand_base_fixed_joint: type fixed, parent left_root_link, child qbhand_base_link, origin xyz=0 0 0 rpy=0 0 0
- added joint qbhand_end_effector_fixed_joint: type fixed, parent qbhand_base_link, child qbhand_end_effector_link, origin xyz=-0.03 0.060 0.142 rpy=-1.57 0 0
- added joint qbhand_index_distal_joint: type revolute, parent qbhand_index_middle_link, child qbhand_index_distal_virtual_link, origin xyz=0.009 0 0 rpy=0 0 0, axis 0 0 -1, limit lower=0.0 upper=0.785 effort=100 velocity=100, mimic joint=qbhand_synergy_joint multiplier=0.785
- added joint qbhand_index_distal_virtual_joint: type revolute, parent qbhand_index_distal_virtual_link, child qbhand_index_distal_link, origin xyz=0.013 0 0 rpy=0 0 0, axis 0 0 -1, limit lower=0.0 upper=0.785 effort=100 velocity=100, mimic joint=qbhand_index_distal_joint multiplier=1.0
- added joint qbhand_index_knuckle_joint: type revolute, parent qbhand_palm_link, child qbhand_index_knuckle_link, origin xyz=-0.02 -0.007 -0.014 rpy=0 3.14 -1.57, axis 0 0 -1, limit lower=-0.524 upper=0.524 effort=100 velocity=100, mimic joint=qbhand_synergy_joint multiplier=0.2
- added joint qbhand_index_middle_joint: type revolute, parent qbhand_index_proximal_link, child qbhand_index_middle_virtual_link, origin xyz=0.017 0 0 rpy=0 0 0, axis 0 0 -1, limit lower=0.0 upper=0.785 effort=100 velocity=100, mimic joint=qbhand_synergy_joint multiplier=0.785
- added joint qbhand_index_middle_virtual_joint: type revolute, parent qbhand_index_middle_virtual_link, child qbhand_index_middle_link, origin xyz=0.013 0 0 rpy=0 0 0, axis 0 0 -1, limit lower=0.0 upper=0.785 effort=100 velocity=100, mimic joint=qbhand_index_middle_joint multiplier=1.0
- added joint qbhand_index_proximal_joint: type revolute, parent qbhand_index_knuckle_link, child qbhand_index_proximal_virtual_link, origin xyz=0.009 0 0 rpy=1.57 0 0, axis 0 0 -1, limit lower=0.0 upper=0.785 effort=100 velocity=100, mimic joint=qbhand_synergy_joint multiplier=0.785
- added joint qbhand_index_proximal_virtual_joint: type revolute, parent qbhand_index_proximal_virtual_link, child qbhand_index_proximal_link, origin xyz=0.013 0 0 rpy=0 0 0, axis 0 0 -1, limit lower=0.0 upper=0.785 effort=100 velocity=100, mimic joint=qbhand_index_proximal_joint multiplier=1.0
- added joint qbhand_little_distal_joint: type revolute, parent qbhand_little_middle_link, child qbhand_little_distal_virtual_link, origin xyz=0.009 0 0 rpy=0 0 0, axis 0 0 -1, limit lower=0.0 upper=0.785 effort=100 velocity=100, mimic joint=qbhand_synergy_joint multiplier=0.785
- added joint qbhand_little_distal_virtual_joint: type revolute, parent qbhand_little_distal_virtual_link, child qbhand_little_distal_link, origin xyz=0.013 0 0 rpy=0 0 0, axis 0 0 -1, limit lower=0.0 upper=0.785 effort=100 velocity=100, mimic joint=qbhand_little_distal_joint multiplier=1.0
- added joint qbhand_little_knuckle_joint: type revolute, parent qbhand_palm_link, child qbhand_little_knuckle_link, origin xyz=0.04 -0.012 -0.014 rpy=0 3.14 -1.57, axis 0 0 -1, limit lower=-0.524 upper=0.524 effort=100 velocity=100, mimic joint=qbhand_synergy_joint multiplier=-0.4
- added joint qbhand_little_middle_joint: type revolute, parent qbhand_little_proximal_link, child qbhand_little_middle_virtual_link, origin xyz=0.009 0 0 rpy=0 0 0, axis 0 0 -1, limit lower=0.0 upper=0.785 effort=100 velocity=100, mimic joint=qbhand_synergy_joint multiplier=0.785
- added joint qbhand_little_middle_virtual_joint: type revolute, parent qbhand_little_middle_virtual_link, child qbhand_little_middle_link, origin xyz=0.013 0 0 rpy=0 0 0, axis 0 0 -1, limit lower=0.0 upper=0.785 effort=100 velocity=100, mimic joint=qbhand_little_middle_joint multiplier=1.0
- added joint qbhand_little_proximal_joint: type revolute, parent qbhand_little_knuckle_link, child qbhand_little_proximal_virtual_link, origin xyz=0.009 0 0 rpy=1.57 0 0, axis 0 0 -1, limit lower=0.0 upper=0.785 effort=100 velocity=100, mimic joint=qbhand_synergy_joint multiplier=0.785
- added joint qbhand_little_proximal_virtual_joint: type revolute, parent qbhand_little_proximal_virtual_link, child qbhand_little_proximal_link, origin xyz=0.013 0 0 rpy=0 0 0, axis 0 0 -1, limit lower=0.0 upper=0.785 effort=100 velocity=100, mimic joint=qbhand_little_proximal_joint multiplier=1.0
- added joint qbhand_middle_distal_joint: type revolute, parent qbhand_middle_middle_link, child qbhand_middle_distal_virtual_link, origin xyz=0.009 0 0 rpy=0 0 0, axis 0 0 -1, limit lower=0.0 upper=0.785 effort=100 velocity=100, mimic joint=qbhand_synergy_joint multiplier=0.785
- added joint qbhand_middle_distal_virtual_joint: type revolute, parent qbhand_middle_distal_virtual_link, child qbhand_middle_distal_link, origin xyz=0.013 0 0 rpy=0 0 0, axis 0 0 -1, limit lower=0.0 upper=0.785 effort=100 velocity=100, mimic joint=qbhand_middle_distal_joint multiplier=1.0
- added joint qbhand_middle_knuckle_joint: type revolute, parent qbhand_palm_link, child qbhand_middle_knuckle_link, origin xyz=0 0 -0.014 rpy=0 3.14 -1.57, axis 0 0 -1, limit lower=-0.524 upper=0.524 effort=100 velocity=100, mimic joint=qbhand_synergy_joint multiplier=0.0
- added joint qbhand_middle_middle_joint: type revolute, parent qbhand_middle_proximal_link, child qbhand_middle_middle_virtual_link, origin xyz=0.017 0 0 rpy=0 0 0, axis 0 0 -1, limit lower=0.0 upper=0.785 effort=100 velocity=100, mimic joint=qbhand_synergy_joint multiplier=0.785
- added joint qbhand_middle_middle_virtual_joint: type revolute, parent qbhand_middle_middle_virtual_link, child qbhand_middle_middle_link, origin xyz=0.013 0 0 rpy=0 0 0, axis 0 0 -1, limit lower=0.0 upper=0.785 effort=100 velocity=100, mimic joint=qbhand_middle_middle_joint multiplier=1.0
- added joint qbhand_middle_proximal_joint: type revolute, parent qbhand_middle_knuckle_link, child qbhand_middle_proximal_virtual_link, origin xyz=0.009 0 0 rpy=1.57 0 0, axis 0 0 -1, limit lower=0.0 upper=0.785 effort=100 velocity=100, mimic joint=qbhand_synergy_joint multiplier=0.785
- added joint qbhand_middle_proximal_virtual_joint: type revolute, parent qbhand_middle_proximal_virtual_link, child qbhand_middle_proximal_link, origin xyz=0.013 0 0 rpy=0 0 0, axis 0 0 -1, limit lower=0.0 upper=0.785 effort=100 velocity=100, mimic joint=qbhand_middle_proximal_joint multiplier=1.0
- added joint qbhand_palm_fixed_joint: type fixed, parent qbhand_base_link, child qbhand_palm_link, origin xyz=0.0045 0.0145 0.144 rpy=1.57 0 3.14
- added joint qbhand_ring_distal_joint: type revolute, parent qbhand_ring_middle_link, child qbhand_ring_distal_virtual_link, origin xyz=0.009 0 0 rpy=0 0 0, axis 0 0 -1, limit lower=0.0 upper=0.785 effort=100 velocity=100, mimic joint=qbhand_synergy_joint multiplier=0.785
- added joint qbhand_ring_distal_virtual_joint: type revolute, parent qbhand_ring_distal_virtual_link, child qbhand_ring_distal_link, origin xyz=0.013 0 0 rpy=0 0 0, axis 0 0 -1, limit lower=0.0 upper=0.785 effort=100 velocity=100, mimic joint=qbhand_ring_distal_joint multiplier=1.0
- added joint qbhand_ring_knuckle_joint: type revolute, parent qbhand_palm_link, child qbhand_ring_knuckle_link, origin xyz=0.02 -0.007 -0.014 rpy=0 3.14 -1.57, axis 0 0 -1, limit lower=-0.524 upper=0.524 effort=100 velocity=100, mimic joint=qbhand_synergy_joint multiplier=-0.2
- added joint qbhand_ring_middle_joint: type revolute, parent qbhand_ring_proximal_link, child qbhand_ring_middle_virtual_link, origin xyz=0.017 0 0 rpy=0 0 0, axis 0 0 -1, limit lower=0.0 upper=0.785 effort=100 velocity=100, mimic joint=qbhand_synergy_joint multiplier=0.785
- added joint qbhand_ring_middle_virtual_joint: type revolute, parent qbhand_ring_middle_virtual_link, child qbhand_ring_middle_link, origin xyz=0.013 0 0 rpy=0 0 0, axis 0 0 -1, limit lower=0.0 upper=0.785 effort=100 velocity=100, mimic joint=qbhand_ring_middle_joint multiplier=1.0
- added joint qbhand_ring_proximal_joint: type revolute, parent qbhand_ring_knuckle_link, child qbhand_ring_proximal_virtual_link, origin xyz=0.009 0 0 rpy=1.57 0 0, axis 0 0 -1, limit lower=0.0 upper=0.785 effort=100 velocity=100, mimic joint=qbhand_synergy_joint multiplier=0.785
- added joint qbhand_ring_proximal_virtual_joint: type revolute, parent qbhand_ring_proximal_virtual_link, child qbhand_ring_proximal_link, origin xyz=0.013 0 0 rpy=0 0 0, axis 0 0 -1, limit lower=0.0 upper=0.785 effort=100 velocity=100, mimic joint=qbhand_ring_proximal_joint multiplier=1.0
- added joint qbhand_synergy_joint: type revolute, parent qbhand_palm_link, child qbhand_synergy_tendon_virtual_link, origin xyz=0 0 0 rpy=0 0 0, axis 0 0 1, limit lower=0.0 upper=1.0 effort=100 velocity=100
- added joint qbhand_thumb_distal_joint: type revolute, parent qbhand_thumb_proximal_link, child qbhand_thumb_distal_virtual_link, origin xyz=0.009 0 0 rpy=0 0 0, axis 0 0 -1, limit lower=0.0 upper=0.785 effort=100 velocity=100, mimic joint=qbhand_synergy_joint multiplier=0.785
- added joint qbhand_thumb_distal_virtual_joint: type revolute, parent qbhand_thumb_distal_virtual_link, child qbhand_thumb_distal_link, origin xyz=0.013 0 0 rpy=0 0 0, axis 0 0 -1, limit lower=0.0 upper=0.785 effort=100 velocity=100, mimic joint=qbhand_thumb_distal_joint multiplier=1.0
- added joint qbhand_thumb_knuckle_joint: type revolute, parent qbhand_palm_link, child qbhand_thumb_knuckle_link, origin xyz=-0.044 -0.0465 0.002 rpy=-1.57 3.14 0.0, axis 0 0 -1, limit lower=0.0 upper=1.571 effort=100 velocity=100, mimic joint=qbhand_synergy_joint multiplier=2.542
- added joint qbhand_thumb_proximal_joint: type revolute, parent qbhand_thumb_knuckle_link, child qbhand_thumb_proximal_virtual_link, origin xyz=0.0255 0.0038 -0.00012 rpy=-2.0 0.0 0.0, axis 0 0 -1, limit lower=0.0 upper=0.785 effort=100 velocity=100, mimic joint=qbhand_synergy_joint multiplier=0.785
- added joint qbhand_thumb_proximal_virtual_joint: type revolute, parent qbhand_thumb_proximal_virtual_link, child qbhand_thumb_proximal_link, origin xyz=0.013 0 0 rpy=0 0 0, axis 0 0 -1, limit lower=0.0 upper=0.785 effort=100 velocity=100, mimic joint=qbhand_thumb_proximal_joint multiplier=1.0

Commit message: added qbhand to curi robot and fixed material problem

File: urdf/curi.urdf (robot description, URDF)
Before this commit: robot curi, 73 links, 72 joints
Links:
- removed link left_root_link
- removed link qbhand_base_link
- removed link qbhand_end_effector_link
- removed link qbhand_index_distal_link
- removed link qbhand_index_distal_virtual_link
- removed link qbhand_index_knuckle_link
- removed link qbhand_index_middle_link
- removed link qbhand_index_middle_virtual_link
- removed link qbhand_index_proximal_link
- removed link qbhand_index_proximal_virtual_link
- removed link qbhand_little_distal_link
- removed link qbhand_little_distal_virtual_link
- removed link qbhand_little_knuckle_link
- removed link qbhand_little_middle_link
- removed link qbhand_little_middle_virtual_link
- removed link qbhand_little_proximal_link
- removed link qbhand_little_proximal_virtual_link
- removed link qbhand_middle_distal_link
- removed link qbhand_middle_distal_virtual_link
- removed link qbhand_middle_knuckle_link
- removed link qbhand_middle_middle_link
- removed link qbhand_middle_middle_virtual_link
- removed link qbhand_middle_proximal_link
- removed link qbhand_middle_proximal_virtual_link
- removed link qbhand_palm_link
- removed link qbhand_ring_distal_link
- removed link qbhand_ring_distal_virtual_link
- removed link qbhand_ring_knuckle_link
- removed link qbhand_ring_middle_link
- removed link qbhand_ring_middle_virtual_link
- removed link qbhand_ring_proximal_link
- removed link qbhand_ring_proximal_virtual_link
- removed link qbhand_synergy_tendon_virtual_link
- removed link qbhand_thumb_distal_link
- removed link qbhand_thumb_distal_virtual_link
- removed link qbhand_thumb_knuckle_link
- removed link qbhand_thumb_proximal_link
- removed link qbhand_thumb_proximal_virtual_link
- added link left_hand_root_link
- added link right_hand_root_link
Joints:
- removed joint panda_end_effector_joint
- removed joint qbhand_base_fixed_joint
- removed joint qbhand_end_effector_fixed_joint
- removed joint qbhand_index_distal_joint
- removed joint qbhand_index_distal_virtual_joint
- removed joint qbhand_index_knuckle_joint
- removed joint qbhand_index_middle_joint
- removed joint qbhand_index_middle_virtual_joint
- removed joint qbhand_index_proximal_joint
- removed joint qbhand_index_proximal_virtual_joint
- removed joint qbhand_little_distal_joint
- removed joint qbhand_little_distal_virtual_joint
- removed joint qbhand_little_knuckle_joint
- removed joint qbhand_little_middle_joint
- removed joint qbhand_little_middle_virtual_joint
- removed joint qbhand_little_proximal_joint
- removed joint qbhand_little_proximal_virtual_joint
- removed joint qbhand_middle_distal_joint
- removed joint qbhand_middle_distal_virtual_joint
- removed joint qbhand_middle_knuckle_joint
- removed joint qbhand_middle_middle_joint
- removed joint qbhand_middle_middle_virtual_joint
- removed joint qbhand_middle_proximal_joint
- removed joint qbhand_middle_proximal_virtual_joint
- removed joint qbhand_palm_fixed_joint
- removed joint qbhand_ring_distal_joint
- removed joint qbhand_ring_distal_virtual_joint
- removed joint qbhand_ring_knuckle_joint
- removed joint qbhand_ring_middle_joint
- removed joint qbhand_ring_middle_virtual_joint
- removed joint qbhand_ring_proximal_joint
- removed joint qbhand_ring_proximal_virtual_joint
- removed joint qbhand_synergy_joint
- removed joint qbhand_thumb_distal_joint
- removed joint qbhand_thumb_distal_virtual_joint
- removed joint qbhand_thumb_knuckle_joint
- removed joint qbhand_thumb_proximal_joint
- removed joint qbhand_thumb_proximal_virtual_joint
- added joint panda_left_end_effector_joint: type fixed, parent panda_left_link7, child left_hand_root_link, origin xyz=0 0 0.107 rpy=0 0 -0.7853981633974483
- added joint panda_right_end_effector_joint: type fixed, parent panda_left_link7, child right_hand_root_link, origin xyz=0 0 0.107 rpy=0 0 -0.7853981633974483

Commit message: added qbhand to curi robot and fixed material problem

File: urdf/curi.urdf (robot description, URDF)
Before this commit: robot curi, 37 links, 36 joints
Links:
- link panda_right_link0: geometry collision mesh filename=../meshes/qbhand/franka/collision/link0.stl; visual mesh filename=../meshes/qbhand/franka/visual/link0.dae
- link panda_right_link1: geometry collision mesh filename=../meshes/qbhand/franka/collision/link1.stl; visual mesh filename=../meshes/qbhand/franka/visual/link1.dae
- link panda_right_link2: geometry collision mesh filename=../meshes/qbhand/franka/collision/link2.stl; visual mesh filename=../meshes/qbhand/franka/visual/link2.dae
- link panda_right_link3: geometry collision mesh filename=../meshes/qbhand/franka/collision/link3.stl; visual mesh filename=../meshes/qbhand/franka/visual/link3.dae
- link panda_right_link4: geometry collision mesh filename=../meshes/qbhand/franka/collision/link4.stl; visual mesh filename=../meshes/qbhand/franka/visual/link4.dae
- link panda_right_link5: geometry collision mesh filename=../meshes/qbhand/franka/collision/link5.stl; visual mesh filename=../meshes/qbhand/franka/visual/link5.dae
- link panda_right_link6: geometry collision mesh filename=../meshes/qbhand/franka/collision/link6.stl; visual mesh filename=../meshes/qbhand/franka/visual/link6.dae
- link panda_right_link7: geometry collision mesh filename=../meshes/qbhand/franka/collision/link7.stl; visual mesh filename=../meshes/qbhand/franka/visual/link7.dae
Joints:
- joint panda_right_end_effector_joint: parent panda_left_link7 -> panda_right_link7
