Commit message: added qbhand to curi robot

File: urdf/curi.urdf (robot description, URDF)
Before this commit: robot curi, 37 links, 36 joints
Links:
- added link left_qbhand_base_link, mass 0.205; collision mesh filename=../meshes/qbhand/flange_iso_04.stl scale=0.001 0.001 0.001; visual mesh filename=../meshes/qbhand/flange_iso_04.stl scale=0.001 0.001 0.001
- added link left_qbhand_end_effector_link
- added link left_qbhand_index_distal_link, mass 0.009; collision mesh filename=../meshes/qbhand/ph_distal_collision.stl scale=0.001 0.001 0.001; visual mesh filename=../meshes/qbhand/ph_distal.stl scale=0.001 0.001 0.001
- added link left_qbhand_index_distal_virtual_link, mass 1e-4
- added link left_qbhand_index_knuckle_link, mass 0.0095; collision mesh filename=../meshes/qbhand/ph_knuckle_collision.stl scale=0.001 0.001 0.001; visual mesh filename=../meshes/qbhand/ph_knuckle.stl scale=0.001 0.001 0.001
- added link left_qbhand_index_middle_link, mass 0.0063; collision mesh filename=../meshes/qbhand/ph_short_collision.stl scale=0.001 0.001 0.001; visual mesh filename=../meshes/qbhand/ph_short.stl scale=0.001 0.001 0.001
- added link left_qbhand_index_middle_virtual_link, mass 1e-4
- added link left_qbhand_index_proximal_link, mass 0.0082; collision mesh filename=../meshes/qbhand/ph_medium_collision.stl scale=0.001 0.001 0.001; visual mesh filename=../meshes/qbhand/ph_medium.stl scale=0.001 0.001 0.001
- added link left_qbhand_index_proximal_virtual_link, mass 1e-4
- added link left_qbhand_little_distal_link, mass 0.009; collision mesh filename=../meshes/qbhand/ph_distal_collision.stl scale=0.001 0.001 0.001; visual mesh filename=../meshes/qbhand/ph_distal.stl scale=0.001 0.001 0.001
- added link left_qbhand_little_distal_virtual_link, mass 1e-4
- added link left_qbhand_little_knuckle_link, mass 0.0095; collision mesh filename=../meshes/qbhand/ph_knuckle_collision.stl scale=0.001 0.001 0.001; visual mesh filename=../meshes/qbhand/ph_knuckle.stl scale=0.001 0.001 0.001
- added link left_qbhand_little_middle_link, mass 0.0063; collision mesh filename=../meshes/qbhand/ph_short_collision.stl scale=0.001 0.001 0.001; visual mesh filename=../meshes/qbhand/ph_short.stl scale=0.001 0.001 0.001
- added link left_qbhand_little_middle_virtual_link, mass 1e-4
- added link left_qbhand_little_proximal_link, mass 0.0063; collision mesh filename=../meshes/qbhand/ph_short_collision.stl scale=0.001 0.001 0.001; visual mesh filename=../meshes/qbhand/ph_short.stl scale=0.001 0.001 0.001
- added link left_qbhand_little_proximal_virtual_link, mass 1e-4
- added link left_qbhand_middle_distal_link, mass 0.009; collision mesh filename=../meshes/qbhand/ph_distal_collision.stl scale=0.001 0.001 0.001; visual mesh filename=../meshes/qbhand/ph_distal.stl scale=0.001 0.001 0.001
- added link left_qbhand_middle_distal_virtual_link, mass 1e-4
- added link left_qbhand_middle_knuckle_link, mass 0.0095; collision mesh filename=../meshes/qbhand/ph_knuckle_collision.stl scale=0.001 0.001 0.001; visual mesh filename=../meshes/qbhand/ph_knuckle.stl scale=0.001 0.001 0.001
- added link left_qbhand_middle_middle_link, mass 0.0063; collision mesh filename=../meshes/qbhand/ph_short_collision.stl scale=0.001 0.001 0.001; visual mesh filename=../meshes/qbhand/ph_short.stl scale=0.001 0.001 0.001
- added link left_qbhand_middle_middle_virtual_link, mass 1e-4
- added link left_qbhand_middle_proximal_link, mass 0.0082; collision mesh filename=../meshes/qbhand/ph_medium_collision.stl scale=0.001 0.001 0.001; visual mesh filename=../meshes/qbhand/ph_medium.stl scale=0.001 0.001 0.001
- added link left_qbhand_middle_proximal_virtual_link, mass 1e-4
- added link left_qbhand_palm_link, mass 0.45; collision mesh filename=../meshes/qbhand/palm_pinch_l.stl scale=0.001 0.001 0.001; visual mesh filename=../meshes/qbhand/palm_pinch_l.stl scale=0.001 0.001 0.001
- added link left_qbhand_ring_distal_link, mass 0.009; collision mesh filename=../meshes/qbhand/ph_distal_collision.stl scale=0.001 0.001 0.001; visual mesh filename=../meshes/qbhand/ph_distal.stl scale=0.001 0.001 0.001
- added link left_qbhand_ring_distal_virtual_link, mass 1e-4
- added link left_qbhand_ring_knuckle_link, mass 0.0095; collision mesh filename=../meshes/qbhand/ph_knuckle_collision.stl scale=0.001 0.001 0.001; visual mesh filename=../meshes/qbhand/ph_knuckle.stl scale=0.001 0.001 0.001
- added link left_qbhand_ring_middle_link, mass 0.0063; collision mesh filename=../meshes/qbhand/ph_short_collision.stl scale=0.001 0.001 0.001; visual mesh filename=../meshes/qbhand/ph_short.stl scale=0.001 0.001 0.001
- added link left_qbhand_ring_middle_virtual_link, mass 1e-4
- added link left_qbhand_ring_proximal_link, mass 0.0082; collision mesh filename=../meshes/qbhand/ph_medium_collision.stl scale=0.001 0.001 0.001; visual mesh filename=../meshes/qbhand/ph_medium.stl scale=0.001 0.001 0.001
- added link left_qbhand_ring_proximal_virtual_link, mass 1e-4
- added link left_qbhand_synergy_tendon_virtual_link, mass 1e-4
- added link left_qbhand_thumb_distal_link, mass 0.009; collision mesh filename=../meshes/qbhand/ph_distal_collision.stl scale=0.001 0.001 0.001; visual mesh filename=../meshes/qbhand/ph_distal.stl scale=0.001 0.001 0.001
- added link left_qbhand_thumb_distal_virtual_link, mass 1e-4
- added link left_qbhand_thumb_knuckle_link, mass 0.01; collision mesh filename=../meshes/qbhand/ph_thumb_l_collision.stl scale=0.001 0.001 0.001; visual mesh filename=../meshes/qbhand/ph_thumb_l.stl scale=0.001 0.001 0.001
- added link left_qbhand_thumb_proximal_link, mass 0.0063; collision mesh filename=../meshes/qbhand/ph_short_collision.stl scale=0.001 0.001 0.001; visual mesh filename=../meshes/qbhand/ph_short.stl scale=0.001 0.001 0.001
- added link left_qbhand_thumb_proximal_virtual_link, mass 1e-4
- added link right_qbhand_base_link, mass 0.45; collision mesh filename=../meshes/qbhand/flange_iso_04.stl scale=0.001 0.001 0.001; visual mesh filename=../meshes/qbhand/flange_iso_04.stl scale=0.001 0.001 0.001
- added link right_qbhand_end_effector_link
- added link right_qbhand_index_distal_link, mass 0.009; collision mesh filename=../meshes/qbhand/ph_distal_collision.stl scale=0.001 0.001 0.001; visual mesh filename=../meshes/qbhand/ph_distal.stl scale=0.001 0.001 0.001
- added link right_qbhand_index_distal_virtual_link, mass 1e-4
- added link right_qbhand_index_knuckle_link, mass 0.0095; collision mesh filename=../meshes/qbhand/ph_knuckle_collision.stl scale=0.001 0.001 0.001; visual mesh filename=../meshes/qbhand/ph_knuckle.stl scale=0.001 0.001 0.001
- added link right_qbhand_index_middle_link, mass 0.0063; collision mesh filename=../meshes/qbhand/ph_short_collision.stl scale=0.001 0.001 0.001; visual mesh filename=../meshes/qbhand/ph_short.stl scale=0.001 0.001 0.001
- added link right_qbhand_index_middle_virtual_link, mass 1e-4
- added link right_qbhand_index_proximal_link, mass 0.0082; collision mesh filename=../meshes/qbhand/ph_medium_collision.stl scale=0.001 0.001 0.001; visual mesh filename=../meshes/qbhand/ph_medium.stl scale=0.001 0.001 0.001
- added link right_qbhand_index_proximal_virtual_link, mass 1e-4
- added link right_qbhand_little_distal_link, mass 0.009; collision mesh filename=../meshes/qbhand/ph_distal_collision.stl scale=0.001 0.001 0.001; visual mesh filename=../meshes/qbhand/ph_distal.stl scale=0.001 0.001 0.001
- added link right_qbhand_little_distal_virtual_link, mass 1e-4
- added link right_qbhand_little_knuckle_link, mass 0.0095; collision mesh filename=../meshes/qbhand/ph_knuckle_collision.stl scale=0.001 0.001 0.001; visual mesh filename=../meshes/qbhand/ph_knuckle.stl scale=0.001 0.001 0.001
- added link right_qbhand_little_middle_link, mass 0.0063; collision mesh filename=../meshes/qbhand/ph_short_collision.stl scale=0.001 0.001 0.001; visual mesh filename=../meshes/qbhand/ph_short.stl scale=0.001 0.001 0.001
- added link right_qbhand_little_middle_virtual_link, mass 1e-4
- added link right_qbhand_little_proximal_link, mass 0.0063; collision mesh filename=../meshes/qbhand/ph_short_collision.stl scale=0.001 0.001 0.001; visual mesh filename=../meshes/qbhand/ph_short.stl scale=0.001 0.001 0.001
- added link right_qbhand_little_proximal_virtual_link, mass 1e-4
- added link right_qbhand_middle_distal_link, mass 0.009; collision mesh filename=../meshes/qbhand/ph_distal_collision.stl scale=0.001 0.001 0.001; visual mesh filename=../meshes/qbhand/ph_distal.stl scale=0.001 0.001 0.001
- added link right_qbhand_middle_distal_virtual_link, mass 1e-4
- added link right_qbhand_middle_knuckle_link, mass 0.0095; collision mesh filename=../meshes/qbhand/ph_knuckle_collision.stl scale=0.001 0.001 0.001; visual mesh filename=../meshes/qbhand/ph_knuckle.stl scale=0.001 0.001 0.001
- added link right_qbhand_middle_middle_link, mass 0.0063; collision mesh filename=../meshes/qbhand/ph_short_collision.stl scale=0.001 0.001 0.001; visual mesh filename=../meshes/qbhand/ph_short.stl scale=0.001 0.001 0.001
- added link right_qbhand_middle_middle_virtual_link, mass 1e-4
- added link right_qbhand_middle_proximal_link, mass 0.0082; collision mesh filename=../meshes/qbhand/ph_medium_collision.stl scale=0.001 0.001 0.001; visual mesh filename=../meshes/qbhand/ph_medium.stl scale=0.001 0.001 0.001
- added link right_qbhand_middle_proximal_virtual_link, mass 1e-4
- added link right_qbhand_palm_link, mass 0.45; collision mesh filename=../meshes/qbhand/palm_pinch_r.stl scale=0.001 0.001 0.001; visual mesh filename=../meshes/qbhand/palm_pinch_r.stl scale=0.001 0.001 0.001
- added link right_qbhand_ring_distal_link, mass 0.009; collision mesh filename=../meshes/qbhand/ph_distal_collision.stl scale=0.001 0.001 0.001; visual mesh filename=../meshes/qbhand/ph_distal.stl scale=0.001 0.001 0.001
- added link right_qbhand_ring_distal_virtual_link, mass 1e-4
- added link right_qbhand_ring_knuckle_link, mass 0.0095; collision mesh filename=../meshes/qbhand/ph_knuckle_collision.stl scale=0.001 0.001 0.001; visual mesh filename=../meshes/qbhand/ph_knuckle.stl scale=0.001 0.001 0.001
- added link right_qbhand_ring_middle_link, mass 0.0063; collision mesh filename=../meshes/qbhand/ph_short_collision.stl scale=0.001 0.001 0.001; visual mesh filename=../meshes/qbhand/ph_short.stl scale=0.001 0.001 0.001
- added link right_qbhand_ring_middle_virtual_link, mass 1e-4
- added link right_qbhand_ring_proximal_link, mass 0.0082; collision mesh filename=../meshes/qbhand/ph_medium_collision.stl scale=0.001 0.001 0.001; visual mesh filename=../meshes/qbhand/ph_medium.stl scale=0.001 0.001 0.001
- added link right_qbhand_ring_proximal_virtual_link, mass 1e-4
- added link right_qbhand_synergy_tendon_virtual_link, mass 1e-4
- added link right_qbhand_thumb_distal_link, mass 0.009; collision mesh filename=../meshes/qbhand/ph_distal_collision.stl scale=0.001 0.001 0.001; visual mesh filename=../meshes/qbhand/ph_distal.stl scale=0.001 0.001 0.001
- added link right_qbhand_thumb_distal_virtual_link, mass 1e-4
- added link right_qbhand_thumb_knuckle_link, mass 0.01; collision mesh filename=../meshes/qbhand/ph_thumb_r_collision.stl scale=0.001 0.001 0.001; visual mesh filename=../meshes/qbhand/ph_thumb_r.stl scale=0.001 0.001 0.001
- added link right_qbhand_thumb_proximal_link, mass 0.0063; collision mesh filename=../meshes/qbhand/ph_short_collision.stl scale=0.001 0.001 0.001; visual mesh filename=../meshes/qbhand/ph_short.stl scale=0.001 0.001 0.001
- added link right_qbhand_thumb_proximal_virtual_link, mass 1e-4
- link panda_right_link0: geometry collision mesh filename=../meshes/franka/collision/link0.stl; visual mesh filename=../meshes/franka/visual/link0.dae
- link panda_right_link1: geometry collision mesh filename=../meshes/franka/collision/link1.stl; visual mesh filename=../meshes/franka/visual/link1.dae
- link panda_right_link2: geometry collision mesh filename=../meshes/franka/collision/link2.stl; visual mesh filename=../meshes/franka/visual/link2.dae
- link panda_right_link3: geometry collision mesh filename=../meshes/franka/collision/link3.stl; visual mesh filename=../meshes/franka/visual/link3.dae
- link panda_right_link4: geometry collision mesh filename=../meshes/franka/collision/link4.stl; visual mesh filename=../meshes/franka/visual/link4.dae
- link panda_right_link5: geometry collision mesh filename=../meshes/franka/collision/link5.stl; visual mesh filename=../meshes/franka/visual/link5.dae
- link panda_right_link6: geometry collision mesh filename=../meshes/franka/collision/link6.stl; visual mesh filename=../meshes/franka/visual/link6.dae
- link panda_right_link7: geometry collision mesh filename=../meshes/franka/collision/link7.stl; visual mesh filename=../meshes/franka/visual/link7.dae
Joints:
- added joint left_qbhand_base_fixed_joint: type fixed, parent left_hand_root_link, child left_qbhand_base_link, origin xyz=0 0 0 rpy=0 0 0
- added joint left_qbhand_end_effector_fixed_joint: type fixed, parent left_qbhand_base_link, child left_qbhand_end_effector_link, origin xyz=-0.03 0.060 0.142 rpy=-1.57 0 0
- added joint left_qbhand_index_distal_joint: type revolute, parent left_qbhand_index_middle_link, child left_qbhand_index_distal_virtual_link, origin xyz=0.009 0 0 rpy=0 0 0, axis 0 0 -1, limit lower=0.0 upper=0.785 effort=100 velocity=100, mimic joint=left_qbhand_synergy_joint multiplier=0.785
- added joint left_qbhand_index_distal_virtual_joint: type revolute, parent left_qbhand_index_distal_virtual_link, child left_qbhand_index_distal_link, origin xyz=0.013 0 0 rpy=0 0 0, axis 0 0 -1, limit lower=0.0 upper=0.785 effort=100 velocity=100, mimic joint=left_qbhand_index_distal_joint multiplier=1.0
- added joint left_qbhand_index_knuckle_joint: type revolute, parent left_qbhand_palm_link, child left_qbhand_index_knuckle_link, origin xyz=-0.02 -0.007 -0.014 rpy=0 3.14 -1.57, axis 0 0 -1, limit lower=-0.524 upper=0.524 effort=100 velocity=100, mimic joint=left_qbhand_synergy_joint multiplier=0.2
- added joint left_qbhand_index_middle_joint: type revolute, parent left_qbhand_index_proximal_link, child left_qbhand_index_middle_virtual_link, origin xyz=0.017 0 0 rpy=0 0 0, axis 0 0 -1, limit lower=0.0 upper=0.785 effort=100 velocity=100, mimic joint=left_qbhand_synergy_joint multiplier=0.785
- added joint left_qbhand_index_middle_virtual_joint: type revolute, parent left_qbhand_index_middle_virtual_link, child left_qbhand_index_middle_link, origin xyz=0.013 0 0 rpy=0 0 0, axis 0 0 -1, limit lower=0.0 upper=0.785 effort=100 velocity=100, mimic joint=left_qbhand_index_middle_joint multiplier=1.0
- added joint left_qbhand_index_proximal_joint: type revolute, parent left_qbhand_index_knuckle_link, child left_qbhand_index_proximal_virtual_link, origin xyz=0.009 0 0 rpy=1.57 0 0, axis 0 0 -1, limit lower=0.0 upper=0.785 effort=100 velocity=100, mimic joint=left_qbhand_synergy_joint multiplier=0.785
- added joint left_qbhand_index_proximal_virtual_joint: type revolute, parent left_qbhand_index_proximal_virtual_link, child left_qbhand_index_proximal_link, origin xyz=0.013 0 0 rpy=0 0 0, axis 0 0 -1, limit lower=0.0 upper=0.785 effort=100 velocity=100, mimic joint=left_qbhand_index_proximal_joint multiplier=1.0
- added joint left_qbhand_little_distal_joint: type revolute, parent left_qbhand_little_middle_link, child left_qbhand_little_distal_virtual_link, origin xyz=0.009 0 0 rpy=0 0 0, axis 0 0 -1, limit lower=0.0 upper=0.785 effort=100 velocity=100, mimic joint=left_qbhand_synergy_joint multiplier=0.785
- added joint left_qbhand_little_distal_virtual_joint: type revolute, parent left_qbhand_little_distal_virtual_link, child left_qbhand_little_distal_link, origin xyz=0.013 0 0 rpy=0 0 0, axis 0 0 -1, limit lower=0.0 upper=0.785 effort=100 velocity=100, mimic joint=left_qbhand_little_distal_joint multiplier=1.0
- added joint left_qbhand_little_knuckle_joint: type revolute, parent left_qbhand_palm_link, child left_qbhand_little_knuckle_link, origin xyz=0.04 -0.012 -0.014 rpy=0 3.14 -1.57, axis 0 0 -1, limit lower=-0.524 upper=0.524 effort=100 velocity=100, mimic joint=left_qbhand_synergy_joint multiplier=-0.4
- added joint left_qbhand_little_middle_joint: type revolute, parent left_qbhand_little_proximal_link, child left_qbhand_little_middle_virtual_link, origin xyz=0.009 0 0 rpy=0 0 0, axis 0 0 -1, limit lower=0.0 upper=0.785 effort=100 velocity=100, mimic joint=left_qbhand_synergy_joint multiplier=0.785
- added joint left_qbhand_little_middle_virtual_joint: type revolute, parent left_qbhand_little_middle_virtual_link, child left_qbhand_little_middle_link, origin xyz=0.013 0 0 rpy=0 0 0, axis 0 0 -1, limit lower=0.0 upper=0.785 effort=100 velocity=100, mimic joint=left_qbhand_little_middle_joint multiplier=1.0
- added joint left_qbhand_little_proximal_joint: type revolute, parent left_qbhand_little_knuckle_link, child left_qbhand_little_proximal_virtual_link, origin xyz=0.009 0 0 rpy=1.57 0 0, axis 0 0 -1, limit lower=0.0 upper=0.785 effort=100 velocity=100, mimic joint=left_qbhand_synergy_joint multiplier=0.785
- added joint left_qbhand_little_proximal_virtual_joint: type revolute, parent left_qbhand_little_proximal_virtual_link, child left_qbhand_little_proximal_link, origin xyz=0.013 0 0 rpy=0 0 0, axis 0 0 -1, limit lower=0.0 upper=0.785 effort=100 velocity=100, mimic joint=left_qbhand_little_proximal_joint multiplier=1.0
- added joint left_qbhand_middle_distal_joint: type revolute, parent left_qbhand_middle_middle_link, child left_qbhand_middle_distal_virtual_link, origin xyz=0.009 0 0 rpy=0 0 0, axis 0 0 -1, limit lower=0.0 upper=0.785 effort=100 velocity=100, mimic joint=left_qbhand_synergy_joint multiplier=0.785
- added joint left_qbhand_middle_distal_virtual_joint: type revolute, parent left_qbhand_middle_distal_virtual_link, child left_qbhand_middle_distal_link, origin xyz=0.013 0 0 rpy=0 0 0, axis 0 0 -1, limit lower=0.0 upper=0.785 effort=100 velocity=100, mimic joint=left_qbhand_middle_distal_joint multiplier=1.0
- added joint left_qbhand_middle_knuckle_joint: type revolute, parent left_qbhand_palm_link, child left_qbhand_middle_knuckle_link, origin xyz=0 0 -0.014 rpy=0 3.14 -1.57, axis 0 0 -1, limit lower=-0.524 upper=0.524 effort=100 velocity=100, mimic joint=left_qbhand_synergy_joint multiplier=0.0
- added joint left_qbhand_middle_middle_joint: type revolute, parent left_qbhand_middle_proximal_link, child left_qbhand_middle_middle_virtual_link, origin xyz=0.017 0 0 rpy=0 0 0, axis 0 0 -1, limit lower=0.0 upper=0.785 effort=100 velocity=100, mimic joint=left_qbhand_synergy_joint multiplier=0.785
- added joint left_qbhand_middle_middle_virtual_joint: type revolute, parent left_qbhand_middle_middle_virtual_link, child left_qbhand_middle_middle_link, origin xyz=0.013 0 0 rpy=0 0 0, axis 0 0 -1, limit lower=0.0 upper=0.785 effort=100 velocity=100, mimic joint=left_qbhand_middle_middle_joint multiplier=1.0
- added joint left_qbhand_middle_proximal_joint: type revolute, parent left_qbhand_middle_knuckle_link, child left_qbhand_middle_proximal_virtual_link, origin xyz=0.009 0 0 rpy=1.57 0 0, axis 0 0 -1, limit lower=0.0 upper=0.785 effort=100 velocity=100, mimic joint=left_qbhand_synergy_joint multiplier=0.785
- added joint left_qbhand_middle_proximal_virtual_joint: type revolute, parent left_qbhand_middle_proximal_virtual_link, child left_qbhand_middle_proximal_link, origin xyz=0.013 0 0 rpy=0 0 0, axis 0 0 -1, limit lower=0.0 upper=0.785 effort=100 velocity=100, mimic joint=left_qbhand_middle_proximal_joint multiplier=1.0
- added joint left_qbhand_palm_fixed_joint: type fixed, parent left_qbhand_base_link, child left_qbhand_palm_link, origin xyz=0.0045 0.0145 0.144 rpy=1.57 0 3.14
- added joint left_qbhand_ring_distal_joint: type revolute, parent left_qbhand_ring_middle_link, child left_qbhand_ring_distal_virtual_link, origin xyz=0.009 0 0 rpy=0 0 0, axis 0 0 -1, limit lower=0.0 upper=0.785 effort=100 velocity=100, mimic joint=left_qbhand_synergy_joint multiplier=0.785
- added joint left_qbhand_ring_distal_virtual_joint: type revolute, parent left_qbhand_ring_distal_virtual_link, child left_qbhand_ring_distal_link, origin xyz=0.013 0 0 rpy=0 0 0, axis 0 0 -1, limit lower=0.0 upper=0.785 effort=100 velocity=100, mimic joint=left_qbhand_ring_distal_joint multiplier=1.0
- added joint left_qbhand_ring_knuckle_joint: type revolute, parent left_qbhand_palm_link, child left_qbhand_ring_knuckle_link, origin xyz=0.02 -0.007 -0.014 rpy=0 3.14 -1.57, axis 0 0 -1, limit lower=-0.524 upper=0.524 effort=100 velocity=100, mimic joint=left_qbhand_synergy_joint multiplier=-0.2
- added joint left_qbhand_ring_middle_joint: type revolute, parent left_qbhand_ring_proximal_link, child left_qbhand_ring_middle_virtual_link, origin xyz=0.017 0 0 rpy=0 0 0, axis 0 0 -1, limit lower=0.0 upper=0.785 effort=100 velocity=100, mimic joint=left_qbhand_synergy_joint multiplier=0.785
- added joint left_qbhand_ring_middle_virtual_joint: type revolute, parent left_qbhand_ring_middle_virtual_link, child left_qbhand_ring_middle_link, origin xyz=0.013 0 0 rpy=0 0 0, axis 0 0 -1, limit lower=0.0 upper=0.785 effort=100 velocity=100, mimic joint=left_qbhand_ring_middle_joint multiplier=1.0
- added joint left_qbhand_ring_proximal_joint: type revolute, parent left_qbhand_ring_knuckle_link, child left_qbhand_ring_proximal_virtual_link, origin xyz=0.009 0 0 rpy=1.57 0 0, axis 0 0 -1, limit lower=0.0 upper=0.785 effort=100 velocity=100, mimic joint=left_qbhand_synergy_joint multiplier=0.785
- added joint left_qbhand_ring_proximal_virtual_joint: type revolute, parent left_qbhand_ring_proximal_virtual_link, child left_qbhand_ring_proximal_link, origin xyz=0.013 0 0 rpy=0 0 0, axis 0 0 -1, limit lower=0.0 upper=0.785 effort=100 velocity=100, mimic joint=left_qbhand_ring_proximal_joint multiplier=1.0
- added joint left_qbhand_synergy_joint: type revolute, parent left_qbhand_palm_link, child left_qbhand_synergy_tendon_virtual_link, origin xyz=0 0 0 rpy=0 0 0, axis 0 0 1, limit lower=0.0 upper=1.0 effort=100 velocity=100
- added joint left_qbhand_thumb_distal_joint: type revolute, parent left_qbhand_thumb_proximal_link, child left_qbhand_thumb_distal_virtual_link, origin xyz=0.009 0 0 rpy=0 0 0, axis 0 0 -1, limit lower=0.0 upper=0.785 effort=100 velocity=100, mimic joint=left_qbhand_synergy_joint multiplier=0.785
- added joint left_qbhand_thumb_distal_virtual_joint: type revolute, parent left_qbhand_thumb_distal_virtual_link, child left_qbhand_thumb_distal_link, origin xyz=0.013 0 0 rpy=0 0 0, axis 0 0 -1, limit lower=0.0 upper=0.785 effort=100 velocity=100, mimic joint=left_qbhand_thumb_distal_joint multiplier=1.0
- added joint left_qbhand_thumb_knuckle_joint: type revolute, parent left_qbhand_palm_link, child left_qbhand_thumb_knuckle_link, origin xyz=-0.044 -0.0465 0.002 rpy=-1.57 3.14 0.0, axis 0 0 -1, limit lower=0.0 upper=1.571 effort=100 velocity=100, mimic joint=left_qbhand_synergy_joint multiplier=2.542
- added joint left_qbhand_thumb_proximal_joint: type revolute, parent left_qbhand_thumb_knuckle_link, child left_qbhand_thumb_proximal_virtual_link, origin xyz=0.0255 0.0038 -0.00012 rpy=-2.0 0.0 0.0, axis 0 0 -1, limit lower=0.0 upper=0.785 effort=100 velocity=100, mimic joint=left_qbhand_synergy_joint multiplier=0.785
- added joint left_qbhand_thumb_proximal_virtual_joint: type revolute, parent left_qbhand_thumb_proximal_virtual_link, child left_qbhand_thumb_proximal_link, origin xyz=0.013 0 0 rpy=0 0 0, axis 0 0 -1, limit lower=0.0 upper=0.785 effort=100 velocity=100, mimic joint=left_qbhand_thumb_proximal_joint multiplier=1.0
- added joint right_qbhand_base_fixed_joint: type fixed, parent right_hand_root_link, child right_qbhand_base_link, origin xyz=0 0 0 rpy=0 0 0
- added joint right_qbhand_end_effector_fixed_joint: type fixed, parent right_qbhand_base_link, child right_qbhand_end_effector_link, origin xyz=-0.03 0.060 0.142 rpy=-1.57 0 0
- added joint right_qbhand_index_distal_joint: type revolute, parent right_qbhand_index_middle_link, child right_qbhand_index_distal_virtual_link, origin xyz=0.009 0 0 rpy=0 0 0, axis 0 0 -1, limit lower=0.0 upper=0.785 effort=100 velocity=100, mimic joint=right_qbhand_synergy_joint multiplier=0.785
- added joint right_qbhand_index_distal_virtual_joint: type revolute, parent right_qbhand_index_distal_virtual_link, child right_qbhand_index_distal_link, origin xyz=0.013 0 0 rpy=0 0 0, axis 0 0 -1, limit lower=0.0 upper=0.785 effort=100 velocity=100, mimic joint=right_qbhand_index_distal_joint multiplier=1.0
- added joint right_qbhand_index_knuckle_joint: type revolute, parent right_qbhand_palm_link, child right_qbhand_index_knuckle_link, origin xyz=-0.02 -0.007 0.014 rpy=0 0 1.57, axis 0 0 -1, limit lower=-0.524 upper=0.524 effort=100 velocity=100, mimic joint=right_qbhand_synergy_joint multiplier=-0.2
- added joint right_qbhand_index_middle_joint: type revolute, parent right_qbhand_index_proximal_link, child right_qbhand_index_middle_virtual_link, origin xyz=0.017 0 0 rpy=0 0 0, axis 0 0 -1, limit lower=0.0 upper=0.785 effort=100 velocity=100, mimic joint=right_qbhand_synergy_joint multiplier=0.785
- added joint right_qbhand_index_middle_virtual_joint: type revolute, parent right_qbhand_index_middle_virtual_link, child right_qbhand_index_middle_link, origin xyz=0.013 0 0 rpy=0 0 0, axis 0 0 -1, limit lower=0.0 upper=0.785 effort=100 velocity=100, mimic joint=right_qbhand_index_middle_joint multiplier=1.0
- added joint right_qbhand_index_proximal_joint: type revolute, parent right_qbhand_index_knuckle_link, child right_qbhand_index_proximal_virtual_link, origin xyz=0.009 0 0 rpy=1.57 0 0, axis 0 0 -1, limit lower=0.0 upper=0.785 effort=100 velocity=100, mimic joint=right_qbhand_synergy_joint multiplier=0.785
- added joint right_qbhand_index_proximal_virtual_joint: type revolute, parent right_qbhand_index_proximal_virtual_link, child right_qbhand_index_proximal_link, origin xyz=0.013 0 0 rpy=0 0 0, axis 0 0 -1, limit lower=0.0 upper=0.785 effort=100 velocity=100, mimic joint=right_qbhand_index_proximal_joint multiplier=1.0
- added joint right_qbhand_little_distal_joint: type revolute, parent right_qbhand_little_middle_link, child right_qbhand_little_distal_virtual_link, origin xyz=0.009 0 0 rpy=0 0 0, axis 0 0 -1, limit lower=0.0 upper=0.785 effort=100 velocity=100, mimic joint=right_qbhand_synergy_joint multiplier=0.785
- added joint right_qbhand_little_distal_virtual_joint: type revolute, parent right_qbhand_little_distal_virtual_link, child right_qbhand_little_distal_link, origin xyz=0.013 0 0 rpy=0 0 0, axis 0 0 -1, limit lower=0.0 upper=0.785 effort=100 velocity=100, mimic joint=right_qbhand_little_distal_joint multiplier=1.0
- added joint right_qbhand_little_knuckle_joint: type revolute, parent right_qbhand_palm_link, child right_qbhand_little_knuckle_link, origin xyz=0.04 -0.012 0.014 rpy=0 0 1.57, axis 0 0 -1, limit lower=-0.524 upper=0.524 effort=100 velocity=100, mimic joint=right_qbhand_synergy_joint multiplier=0.4
- added joint right_qbhand_little_middle_joint: type revolute, parent right_qbhand_little_proximal_link, child right_qbhand_little_middle_virtual_link, origin xyz=0.009 0 0 rpy=0 0 0, axis 0 0 -1, limit lower=0.0 upper=0.785 effort=100 velocity=100, mimic joint=right_qbhand_synergy_joint multiplier=0.785
- added joint right_qbhand_little_middle_virtual_joint: type revolute, parent right_qbhand_little_middle_virtual_link, child right_qbhand_little_middle_link, origin xyz=0.013 0 0 rpy=0 0 0, axis 0 0 -1, limit lower=0.0 upper=0.785 effort=100 velocity=100, mimic joint=right_qbhand_little_middle_joint multiplier=1.0
- added joint right_qbhand_little_proximal_joint: type revolute, parent right_qbhand_little_knuckle_link, child right_qbhand_little_proximal_virtual_link, origin xyz=0.009 0 0 rpy=1.57 0 0, axis 0 0 -1, limit lower=0.0 upper=0.785 effort=100 velocity=100, mimic joint=right_qbhand_synergy_joint multiplier=0.785
- added joint right_qbhand_little_proximal_virtual_joint: type revolute, parent right_qbhand_little_proximal_virtual_link, child right_qbhand_little_proximal_link, origin xyz=0.013 0 0 rpy=0 0 0, axis 0 0 -1, limit lower=0.0 upper=0.785 effort=100 velocity=100, mimic joint=right_qbhand_little_proximal_joint multiplier=1.0
- added joint right_qbhand_middle_distal_joint: type revolute, parent right_qbhand_middle_middle_link, child right_qbhand_middle_distal_virtual_link, origin xyz=0.009 0 0 rpy=0 0 0, axis 0 0 -1, limit lower=0.0 upper=0.785 effort=100 velocity=100, mimic joint=right_qbhand_synergy_joint multiplier=0.785
- added joint right_qbhand_middle_distal_virtual_joint: type revolute, parent right_qbhand_middle_distal_virtual_link, child right_qbhand_middle_distal_link, origin xyz=0.013 0 0 rpy=0 0 0, axis 0 0 -1, limit lower=0.0 upper=0.785 effort=100 velocity=100, mimic joint=right_qbhand_middle_distal_joint multiplier=1.0
- added joint right_qbhand_middle_knuckle_joint: type revolute, parent right_qbhand_palm_link, child right_qbhand_middle_knuckle_link, origin xyz=0 0 0.014 rpy=0 0 1.57, axis 0 0 -1, limit lower=-0.524 upper=0.524 effort=100 velocity=100, mimic joint=right_qbhand_synergy_joint multiplier=0.0
- added joint right_qbhand_middle_middle_joint: type revolute, parent right_qbhand_middle_proximal_link, child right_qbhand_middle_middle_virtual_link, origin xyz=0.017 0 0 rpy=0 0 0, axis 0 0 -1, limit lower=0.0 upper=0.785 effort=100 velocity=100, mimic joint=right_qbhand_synergy_joint multiplier=0.785
- added joint right_qbhand_middle_middle_virtual_joint: type revolute, parent right_qbhand_middle_middle_virtual_link, child right_qbhand_middle_middle_link, origin xyz=0.013 0 0 rpy=0 0 0, axis 0 0 -1, limit lower=0.0 upper=0.785 effort=100 velocity=100, mimic joint=right_qbhand_middle_middle_joint multiplier=1.0
- added joint right_qbhand_middle_proximal_joint: type revolute, parent right_qbhand_middle_knuckle_link, child right_qbhand_middle_proximal_virtual_link, origin xyz=0.009 0 0 rpy=1.57 0 0, axis 0 0 -1, limit lower=0.0 upper=0.785 effort=100 velocity=100, mimic joint=right_qbhand_synergy_joint multiplier=0.785
- added joint right_qbhand_middle_proximal_virtual_joint: type revolute, parent right_qbhand_middle_proximal_virtual_link, child right_qbhand_middle_proximal_link, origin xyz=0.013 0 0 rpy=0 0 0, axis 0 0 -1, limit lower=0.0 upper=0.785 effort=100 velocity=100, mimic joint=right_qbhand_middle_proximal_joint multiplier=1.0
- added joint right_qbhand_palm_fixed_joint: type fixed, parent right_qbhand_base_link, child right_qbhand_palm_link, origin xyz=-0.0045 0.0145 0.144 rpy=1.57 0 0
- added joint right_qbhand_ring_distal_joint: type revolute, parent right_qbhand_ring_middle_link, child right_qbhand_ring_distal_virtual_link, origin xyz=0.009 0 0 rpy=0 0 0, axis 0 0 -1, limit lower=0.0 upper=0.785 effort=100 velocity=100, mimic joint=right_qbhand_synergy_joint multiplier=0.785
- added joint right_qbhand_ring_distal_virtual_joint: type revolute, parent right_qbhand_ring_distal_virtual_link, child right_qbhand_ring_distal_link, origin xyz=0.013 0 0 rpy=0 0 0, axis 0 0 -1, limit lower=0.0 upper=0.785 effort=100 velocity=100, mimic joint=right_qbhand_ring_distal_joint multiplier=1.0
- added joint right_qbhand_ring_knuckle_joint: type revolute, parent right_qbhand_palm_link, child right_qbhand_ring_knuckle_link, origin xyz=0.02 -0.007 0.014 rpy=0 0 1.57, axis 0 0 -1, limit lower=-0.524 upper=0.524 effort=100 velocity=100, mimic joint=right_qbhand_synergy_joint multiplier=0.2
- added joint right_qbhand_ring_middle_joint: type revolute, parent right_qbhand_ring_proximal_link, child right_qbhand_ring_middle_virtual_link, origin xyz=0.017 0 0 rpy=0 0 0, axis 0 0 -1, limit lower=0.0 upper=0.785 effort=100 velocity=100, mimic joint=right_qbhand_synergy_joint multiplier=0.785
- added joint right_qbhand_ring_middle_virtual_joint: type revolute, parent right_qbhand_ring_middle_virtual_link, child right_qbhand_ring_middle_link, origin xyz=0.013 0 0 rpy=0 0 0, axis 0 0 -1, limit lower=0.0 upper=0.785 effort=100 velocity=100, mimic joint=right_qbhand_ring_middle_joint multiplier=1.0
- added joint right_qbhand_ring_proximal_joint: type revolute, parent right_qbhand_ring_knuckle_link, child right_qbhand_ring_proximal_virtual_link, origin xyz=0.009 0 0 rpy=1.57 0 0, axis 0 0 -1, limit lower=0.0 upper=0.785 effort=100 velocity=100, mimic joint=right_qbhand_synergy_joint multiplier=0.785
- added joint right_qbhand_ring_proximal_virtual_joint: type revolute, parent right_qbhand_ring_proximal_virtual_link, child right_qbhand_ring_proximal_link, origin xyz=0.013 0 0 rpy=0 0 0, axis 0 0 -1, limit lower=0.0 upper=0.785 effort=100 velocity=100, mimic joint=right_qbhand_ring_proximal_joint multiplier=1.0
- added joint right_qbhand_synergy_joint: type revolute, parent right_qbhand_palm_link, child right_qbhand_synergy_tendon_virtual_link, origin xyz=0 0 0 rpy=0 0 0, axis 0 0 1, limit lower=0.0 upper=1.0 effort=100 velocity=100
- added joint right_qbhand_thumb_distal_joint: type revolute, parent right_qbhand_thumb_proximal_link, child right_qbhand_thumb_distal_virtual_link, origin xyz=0.009 0 0 rpy=0 0 0, axis 0 0 -1, limit lower=0.0 upper=0.785 effort=100 velocity=100, mimic joint=right_qbhand_synergy_joint multiplier=0.785
- added joint right_qbhand_thumb_distal_virtual_joint: type revolute, parent right_qbhand_thumb_distal_virtual_link, child right_qbhand_thumb_distal_link, origin xyz=0.013 0 0 rpy=0 0 0, axis 0 0 -1, limit lower=0.0 upper=0.785 effort=100 velocity=100, mimic joint=right_qbhand_thumb_distal_joint multiplier=1.0
- added joint right_qbhand_thumb_knuckle_joint: type revolute, parent right_qbhand_palm_link, child right_qbhand_thumb_knuckle_link, origin xyz=-0.044 -0.0465 -0.002 rpy=-1.57 3.14 0.0, axis 0 0 -1, limit lower=0.0 upper=1.571 effort=100 velocity=100, mimic joint=right_qbhand_synergy_joint multiplier=2.542
- added joint right_qbhand_thumb_proximal_joint: type revolute, parent right_qbhand_thumb_knuckle_link, child right_qbhand_thumb_proximal_virtual_link, origin xyz=0.0255 -0.0038 -0.00012 rpy=-1.1415 0.0 0.0, axis 0 0 -1, limit lower=0.0 upper=0.785 effort=100 velocity=100, mimic joint=right_qbhand_synergy_joint multiplier=0.785
- added joint right_qbhand_thumb_proximal_virtual_joint: type revolute, parent right_qbhand_thumb_proximal_virtual_link, child right_qbhand_thumb_proximal_link, origin xyz=0.013 0 0 rpy=0 0 0, axis 0 0 -1, limit lower=0.0 upper=0.785 effort=100 velocity=100, mimic joint=right_qbhand_thumb_proximal_joint multiplier=1.0
